File: brd/Turntable.brd (EAGLE design)
At the start: 100 x 80 mm, 115 parts, among them CON1 Pannel, CON2 CAN, CON3 Turntable, CON4 STEPPER_CON, CON5 STEPPER_CON, CON8 SPK, IC1 7805, IC2 LM393N, J1 MiniStp2, J10 MiniStp1, Q1 BS170, SW1 EC12E_SW, U2 LED NANO, X1 AK500/2+M, X2 AK500/2+M, X3 MAB 5SH Conrad: 738247 - VQ, X4 AK500/2+M, X5 Reichelt MEBP 8-8S

Commit message: Final Version 1.0
Parts:
- added JP20, JP21: Mode, adafruit:1X03-CLEANBIG
- JP4, JP8: value EnabMod -> Enab; device SparkFun-Connectors:1X02 -> adafruit:1X03-CLEANBIG
- R19: value 10K -> Opt
- moved JP8 0.63 mm to (27.3, 64.8)
Connections:
- new net N$32: JP21.3, U$1.SLEEP
- new net N$33: JP20.3, U$5.SLEEP
- net +5V: now also JP4.1, JP8.1
- net ENAB_STEP: now also JP20.1, JP4.3; no longer JP4.1
- net N$30: now also JP20.2; no longer U$5.SLEEP
- net N$46: now also JP21.2; no longer U$1.SLEEP
- net SX/CS_CAN: now also JP21.1, JP8.3; no longer JP8.1
Routing:
- net SX/CS_CAN: track 87.9 -> 102.7 mm
- net DCC/SX: track 86.0 -> 99.3 mm
- net ENAB_STEP: track 100.7 -> 113.7 mm, vias 1 -> 2
- net D12: track 51.3 -> 58.2 mm
- net SCL: track 157.3 -> 162.6 mm
- net N$33: track 0.00 -> 4.23 mm
- net N$30: track 2.55 -> 6.64 mm
- net +5V: track 399.8 -> 403.7 mm
- net D11: track 69.4 -> 73.2 mm
- net N$32: track 0.00 -> 3.59 mm
- net N$25: track 3.27 -> 6.64 mm
- net N$46: track 2.67 -> 6.01 mm
- net N$45: track 3.19 -> 6.01 mm
- net N$47: track 51.2 -> 48.4 mm
- net N$5: track 153.6 -> 156.0 mm
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